Commit message: Stair Climbing Successfully

File: src/vaccum_description/urdf/vaccum.ros2_control.xacro (robot description, xacro)
@@ -1,3 +1,7 @@
 <?xml version="1.0"?>
+<!-- controller_joint_names:
+['', 'front_left_wheel_joint', 'front_right_wheel_joint',
+'rear_left_wheel_joint',
+'left_middle_arm_to_base_joint', 'left_arm_joint', 'right_middle_arm_to_base_joint', 'right_arm_joint', ] -->
 <robot xmlns:xacro="http://www.ros.org/wiki/xacro">
   <xacro:macro name="vaccum_ros2_control" params="name prefix">
@@ -26,4 +30,24 @@
         <state_interface name="position"/>
       </joint>
+      <joint name="left_middle_arm_to_base_joint">
+        <command_interface name="position"/>
+        <state_interface name="velocity"/>
+        <state_interface name="position"/>
+      </joint>
+      <joint name="left_arm_joint">
+        <command_interface name="position"/>
+        <state_interface name="velocity"/>
+        <state_interface name="position"/>
+      </joint>
+      <joint name="right_middle_arm_to_base_joint">
+        <command_interface name="position"/>
+        <state_interface name="velocity"/>
+        <state_interface name="position"/>
+      </joint>
+      <joint name="right_arm_joint">
+        <command_interface name="position"/>
+        <state_interface name="velocity"/>
+        <state_interface name="position"/>
+      </joint>
     </ros2_control>
   </xacro:macro>

File: src/vaccum_description/urdf/vaccum_description.urdf.xacro (robot description, xacro)
@@ -415,4 +415,5 @@
     <axis
       xyz="0 0 -1" />
+      <limit effort="99.0" velocity="99.0" />
   </joint>
   <link
@@ -468,4 +469,5 @@
     <axis
       xyz="0 0 -1" />
+      <limit effort="99.0" velocity="99.0" />
   </joint>
   <link
@@ -521,4 +523,5 @@
     <axis
       xyz="0 0 -1" />
+      <limit effort="99.0" velocity="99.0" />
   </joint>
   <link
@@ -574,4 +577,5 @@
     <axis
       xyz="0 0 -1" />
+      <limit effort="99.0" velocity="99.0" />
   </joint>
   </xacro:macro>
