Commit message: Control Setup Done

File: src/vaccum_description/urdf/vaccum_description.urdf.xacro (robot description, xacro)
@@ -5,574 +5,574 @@
 <robot xmlns:xacro="http://www.ros.org/wiki/xacro">
   <xacro:macro name="vaccum" params="parent prefix *origin">
-    <link
-      name="base_link">
-      <inertial>
-        <origin
-          xyz="-0.020239 0.00031106 0.034044"
-          rpy="0 0 0" />
-        <mass
-          value="1.4598" />
-        <inertia
-          ixx="0.0019201"
-          ixy="-1.9441E-06"
-          ixz="1.5768E-06"
-          iyy="0.0036049"
-          iyz="-5.9889E-08"
-          izz="0.0047447" />
-      </inertial>
-      <visual>
-        <origin
-          xyz="0 0 0"
-          rpy="0 0 0" />
-        <geometry>
-          <mesh
-            filename="$(find vaccum_description)/meshes/base_link.STL" />
-        </geometry>
-        <material
-          name="">
-          <color
-            rgba="0.79608 0.79608 0.79608 1" />
-        </material>
-      </visual>
-      <collision>
-        <origin
-          xyz="0 0 0"
-          rpy="0 0 0" />
-        <geometry>
-          <mesh
-            filename="$(find vaccum_description)/meshes/base_link.STL" />
-        </geometry>
-      </collision>
-    </link>
-    <link
-      name="front_left_wheel">
-      <inertial>
-        <origin
-          xyz="4.2207E-06 4.885E-15 -0.0089401"
-          rpy="0 0 0" />
-        <mass
-          value="0.013528" />
-        <inertia
-          ixx="2.2635E-06"
-          ixy="-7.79E-20"
-          ixz="1.0999E-10"
-          iyy="2.2633E-06"
-          iyz="1.1804E-19"
-          izz="3.9268E-06" />
-      </inertial>
-      <visual>
-        <origin
-          xyz="0 0 0"
-          rpy="0 0 0" />
-        <geometry>
-          <mesh
-            filename="$(find vaccum_description)/meshes/front_left_wheel.STL" />
-        </geometry>
-        <material
-          name="">
-          <color
-            rgba="0.79608 0.82353 0.93725 1" />
-        </material>
-      </visual>
-      <collision>
-        <origin
-          xyz="0 0 0"
-          rpy="0 0 0" />
-        <geometry>
-          <mesh
-            filename="$(find vaccum_description)/meshes/front_left_wheel.STL" />
-        </geometry>
-      </collision>
-    </link>
-    <joint
-      name="front_left_wheel_joint"
-      type="continuous">
-      <origin
-        xyz="0.06336 0.063002 0.0075"
-        rpy="1.5708 0 0" />
-      <parent
-        link="base_link" />
-      <child
-        link="front_left_wheel" />
-      <axis
-        xyz="0 0 -1" />
-    </joint>
-    <link
-      name="front_right_wheel">
-      <inertial>
-        <origin
-          xyz="0.124340591481911 4.74620343027254E-15 0.00894007340577986"
-          rpy="0 0 0" />
-        <mass
-          value="0.0135281025569348" />
-        <inertia
-          ixx="2.26349850351656E-06"
-          ixy="-4.85019556681031E-20"
-          ixz="1.09985013202205E-10"
-          iyy="2.26334994628094E-06"
-          iyz="1.20786707459227E-20"
-          izz="3.9267511636668E-06" />
-      </inertial>
-      <visual>
-        <origin
-          xyz="0 0 0"
-          rpy="0 0 0" />
-        <geometry>
-          <mesh
-            filename="$(find vaccum_description)/meshes/front_right_wheel.STL" />
-        </geometry>
-        <material
-          name="">
-          <color
-            rgba="0.796078431372549 0.823529411764706 0.937254901960784 1" />
-        </material>
-      </visual>
-      <collision>
-        <origin
-          xyz="0 0 0"
-          rpy="0 0 0" />
-        <geometry>
-          <mesh
-            filename="$(find vaccum_description)/meshes/front_right_wheel.STL" />
-        </geometry>
-      </collision>
-    </link>
-    <joint
-      name="front_right_wheel_joint"
-      type="continuous">
-      <origin
-        xyz="-0.060985 -0.062997 0.0075"
-        rpy="1.5708 0 0" />
-      <parent
-        link="base_link" />
-      <child
-        link="front_right_wheel" />
-      <axis
-        xyz="0 0 1" />
-    </joint>
-    <link
-      name="rear_left_wheel">
-      <inertial>
-        <origin
-          xyz="4.22068515629204E-06 4.75661177112841E-15 -0.00894007340577976"
-          rpy="0 0 0" />
-        <mass
-          value="0.0135281025569348" />
-        <inertia
-          ixx="2.26349850351647E-06"
-          ixy="1.0398033549131E-19"
-          ixz="1.09985013393305E-10"
-          iyy="2.26334994628079E-06"
-          iyz="1.22371024055836E-19"
-          izz="3.9267511636666E-06" />
-      </inertial>
-      <visual>
-        <origin
-          xyz="0 0 0"
-          rpy="0 0 0" />
-        <geometry>
-          <mesh
-            filename="$(find vaccum_description)/meshes/rear_left_wheel.STL" />
-        </geometry>
-        <material
-          name="">
-          <color
-            rgba="0.796078431372549 0.823529411764706 0.937254901960784 1" />
-        </material>
-      </visual>
-      <collision>
-        <origin
-          xyz="0 0 0"
-          rpy="0 0 0" />
-        <geometry>
-          <mesh
-            filename="$(find vaccum_description)/meshes/rear_left_wheel.STL" />
-        </geometry>
-      </collision>
-    </link>
-    <joint
-      name="rear_left_wheel_joint"
-      type="continuous">
-      <origin
-        xyz="-0.060985 0.063002 0.0075"
-        rpy="1.5708 0 0" />
-      <parent
-        link="base_link" />
-      <child
-        link="rear_left_wheel" />
-      <axis
-        xyz="0 0 -1" />
-    </joint>
-    <link
-      name="rear_right_wheel">
-      <inertial>
-        <origin
-          xyz="-4.2207E-06 4.9925E-15 0.0089401"
-          rpy="0 0 0" />
-        <mass
-          value="0.013528" />
-        <inertia
-          ixx="2.2635E-06"
-          ixy="-8.4853E-20"
-          ixz="1.0999E-10"
-          iyy="2.2633E-06"
-          iyz="1.2044E-21"
-          izz="3.9268E-06" />
-      </inertial>
-      <visual>
-        <origin
-          xyz="0 0 0"
-          rpy="0 0 0" />
-        <geometry>
-          <mesh
-            filename="$(find vaccum_description)/meshes/rear_right_wheel.STL" />
-        </geometry>
-        <material
-          name="">
-          <color
-            rgba="0.79608 0.82353 0.93725 1" />
-        </material>
-      </visual>
-      <collision>
-        <origin
-          xyz="0 0 0"
-          rpy="0 0 0" />
-        <geometry>
-          <mesh
-            filename="$(find vaccum_description)/meshes/rear_right_wheel.STL" />
-        </geometry>
-      </collision>
-    </link>
-    <joint
-      name="rear_right_wheel_joint"
-      type="continuous">
-      <origin
-        xyz="-0.0609849382460916 -0.0629970469534928 0.00749999999999469"
-        rpy="1.5707963267949 0 0" />
-      <parent
-        link="base_link" />
-      <child
-        link="rear_right_wheel" />
-      <axis
-        xyz="0 0 1" />
-    </joint>
-    <link
-      name="camera">
-      <inertial>
-        <origin
-          xyz="-0.00998796510467402 0.00185487708558293 -1.97498793444439E-06"
-          rpy="0 0 0" />
-        <mass
-          value="0.00251010214351842" />
-        <inertia
-          ixx="1.4088701772609E-07"
-          ixy="4.33759503016402E-09"
-          ixz="-4.63200736869362E-12"
-          iyy="8.82173300651778E-08"
-          iyz="-3.32907116776564E-11"
-          izz="9.33512132066443E-08" />
-      </inertial>
-      <visual>
-        <origin
-          xyz="0 0 0"
-          rpy="0 0 0" />
-        <geometry>
-          <mesh
-            filename="$(find vaccum_description)/meshes/camera.STL" />
-        </geometry>
-        <material
-          name="">
-          <color
-            rgba="0.752941176470588 0.752941176470588 0.752941176470588 1" />
-        </material>
-      </visual>
-      <collision>
-        <origin
-          xyz="0 0 0"
-          rpy="0 0 0" />
-        <geometry>
-          <mesh
-            filename="$(find vaccum_description)/meshes/camera.STL" />
-        </geometry>
-      </collision>
-    </link>
-    <joint
-      name="camerajoint"
-      type="fixed">
-      <origin
-        xyz="0.10632 0 0.05433"
-        rpy="1.5708 0 0" />
-      <parent
-        link="base_link" />
-      <child
-        link="camera" />
-      <axis
-        xyz="0 0 0" />
-    </joint>
-    <link
-      name="lidar">
-      <inertial>
-        <origin
-          xyz="-0.0051082 0.00096996 8.8966E-08"
-          rpy="0 0 0" />
-        <mass
-          value="0.083344" />
-        <inertia
-          ixx="2.4035E-05"
-          ixy="-1.2606E-06"
-          ixz="-6.5531E-10"
-          iyy="5.1914E-05"
-          iyz="-1.2872E-11"
-          izz="3.3173E-05" />
-      </inertial>
-      <visual>
-        <origin
-          xyz="0 0 0"
-          rpy="0 0 0" />
-        <geometry>
-          <mesh
-            filename="$(find vaccum_description)/meshes/lidar.STL" />
-        </geometry>
-        <material
-          name="">
-          <color
-            rgba="1 1 1 1" />
-        </material>
-      </visual>
-      <collision>
-        <origin
-          xyz="0 0 0"
-          rpy="0 0 0" />
-        <geometry>
-          <mesh
-            filename="$(find vaccum_description)/meshes/lidar.STL" />
-        </geometry>
-      </collision>
-    </link>
-    <joint
-      name="lidar_joint"
-      type="fixed">
-      <origin
-        xyz="-6.0126E-05 0 0.07633"
-        rpy="1.5708 0 1.5708" />
-      <parent
-        link="base_link" />
-      <child
-        link="lidar" />
-      <axis
-        xyz="0 0 0" />
-    </joint>
-    <link
-      name="left_middle_arm">
-      <inertial>
-        <origin
-          xyz="-0.0925422766892284 -0.00809825655008783 -0.00375285653305618"
-          rpy="0 0 0" />
-        <mass
-          value="0.157769108071277" />
-        <inertia
-          ixx="8.59338792255128E-05"
-          ixy="5.40150112353752E-08"
-          ixz="-5.22234310271608E-06"
-          iyy="0.0008635371367084"
-          iyz="3.64966292115922E-09"
-          izz="0.000947374926548457" />
-      </inertial>
-      <visual>
-        <origin
-          xyz="0 0 0"
-          rpy="0 0 0" />
-        <geometry>
-          <mesh
-            filename="$(find vaccum_description)/meshes/left_middle_arm.STL" />
-        </geometry>
-        <material
-          name="">
-          <color
-            rgba="0.792156862745098 0.819607843137255 0.933333333333333 1" />
-        </material>
-      </visual>
-      <collision>
-        <origin
-          xyz="0 0 0"
-          rpy="0 0 0" />
-        <geometry>
-          <mesh
-            filename="$(find vaccum_description)/meshes/left_middle_arm.STL" />
-        </geometry>
-      </collision>
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
Commit message: Camera Simulation setup done:

File: src/vaccum_description/urdf/vaccum_description.urdf.xacro (robot description, xacro)
@@ -310,4 +310,36 @@
       xyz="0 0 0" />
   </joint>
+  <!-- Camera Optical link -->
+    <joint name="camera_optical_joint" type="fixed">
+        <parent link="camera"/>
+        <child link="camera_link_optical"/>
+        <origin xyz="0 0 0" rpy="0 0 0"/>
+    </joint>
+    <link name="camera_link_optical"></link>
+    <!-- Camera Gazebo Sensor Plugin -->
+    <gazebo reference="camera">
+        <material>Gazebo/Black</material>
+        <sensor name="camera" type="camera">
+            <pose> 0 0 0 -1.5707 0 0 </pose>
+            <always_on>true</always_on>
+            <visualize>true</visualize>
+            <update_rate>30</update_rate>
+            <topic>camera/image</topic>
+            <gz_frame_id>camera_link_optical</gz_frame_id>
+            <camera>
+                <camera_info_topic>camera/camera_info</camera_info_topic>
+                <horizontal_fov>1.089</horizontal_fov>
+                <image>
+                    <format>R8G8B8</format>
+                    <width>640</width>
+                    <height>480</height>
+                </image>
+                <clip>
+                    <near>0.05</near>
+                    <far>8.0</far>
+                </clip>
+            </camera>
+        </sensor>
+    </gazebo>
   <link
     name="lidar">
@@ -363,4 +395,28 @@
       xyz="0 0 0" />
   </joint>
+<gazebo reference="lidar">
+        <material>Gazebo/Grey</material>
+        <sensor name="laser" type="gpu_lidar">
+            <pose> 0 0 0 0 0 0 </pose>
+            <always_on>true</always_on>
+            <visualize>true</visualize>
+            <update_rate>10</update_rate>
+            <topic>scan</topic>
+            <gz_frame_id>lidar</gz_frame_id>
+            <lidar>
+                <scan>
+                    <horizontal>
+                        <samples>360</samples>
+                        <min_angle>-3.14</min_angle>
+                        <max_angle>3.14</max_angle>
+                    </horizontal>
+                </scan>
+                <range>
+                    <min>0.3</min>
+                    <max>12</max>
+                </range>
+            </lidar>
+        </sensor>
+    </gazebo>
   <link
     name="left_middle_arm">

Commit message: robot color changed

File: src/vaccum_description/urdf/vaccum_description.urdf.xacro (robot description, xacro)
@@ -30,7 +30,7 @@
       </geometry>
       <material
-        name="">
-        <color
-          rgba="0.796078431372549 0.796078431372549 0.796078431372549 1" />
+        name="yellow">
+        <color
+          rgba="0.8 0.8 0.0 1.0" />
       </material>
     </visual>
@@ -70,7 +70,7 @@
       </geometry>
       <material
-        name="">
-        <color
-          rgba="0.796078431372549 0.823529411764706 0.937254901960784 1" />
+        name="black">
+        <color
+          rgba="0 0 0 1" />
       </material>
     </visual>
@@ -122,8 +122,8 @@
           filename="file://$(find vaccum_description)/meshes/front_right_wheel.STL" />
       </geometry>
-      <material
-        name="">
-        <color
-          rgba="0.796078431372549 0.823529411764706 0.937254901960784 1" />
+     <material
+        name="black">
+        <color
+          rgba="0 0 0 1" />
       </material>
     </visual>
@@ -176,7 +176,7 @@
       </geometry>
       <material
-        name="">
-        <color
-          rgba="0.796078431372549 0.823529411764706 0.937254901960784 1" />
+        name="black">
+        <color
+          rgba="0 0 0 1" />
       </material>
     </visual>
@@ -228,8 +228,8 @@
           filename="file://$(find vaccum_description)/meshes/rear_right_wheel.STL" />
       </geometry>
-      <material
-        name="">
-        <color
-          rgba="0.796078431372549 0.823529411764706 0.937254901960784 1" />
+     <material
+        name="black">
+        <color
+          rgba="0 0 0 1" />
       </material>
     </visual>
@@ -281,8 +281,8 @@
           filename="file://$(find vaccum_description)/meshes/camera.STL" />
       </geometry>
-      <material
-        name="">
-        <color
-          rgba="0.752941176470588 0.752941176470588 0.752941176470588 1" />
+    <material
+        name="black">
+        <color
+          rgba="0 0 0 1" />
       </material>
     </visual>
@@ -366,8 +366,8 @@
           filename="file://$(find vaccum_description)/meshes/lidar.STL" />
       </geometry>
-      <material
-        name="">
-        <color
-          rgba="1 1 1 1" />
+     <material
+        name="black">
+        <color
+          rgba="0 0 0 1" />
       </material>
     </visual>
@@ -444,7 +444,7 @@
       </geometry>
       <material
-        name="">
-        <color
-          rgba="0.792156862745098 0.819607843137255 0.933333333333333 1" />
+        name="orange">
+        <color
+          rgba="1 0.647058823529412 0 1" />
       </material>
     </visual>
@@ -498,7 +498,7 @@
       </geometry>
       <material
-        name="">
-        <color
-          rgba="0.752941176470588 0.752941176470588 0.752941176470588 1" />
+        name="black">
+        <color
+          rgba="0 0 0 1" />
       </material>
     </visual>
@@ -551,8 +551,8 @@
           filename="file://$(find vaccum_description)/meshes/right_middle_arm.STL" />
       </geometry>
-      <material
-        name="">
-        <color
-          rgba="0.792156862745098 0.819607843137255 0.933333333333333 1" />
+       <material
+        name="orange">
+        <color
+          rgba="1 0.647058823529412 0 1" />
       </material>
     </visual>
@@ -606,7 +606,7 @@
       </geometry>
       <material
-        name="">
-        <color
-          rgba="0.752941176470588 0.752941176470588 0.752941176470588 1" />
+        name="black">
+        <color
+          rgba="0 0 0 1" />
       </material>
     </visual>

Commit message: Lidar Sensor Simulation Setup Done

File: src/vaccum_description/urdf/vaccum_description.urdf.xacro (robot description, xacro)
@@ -395,5 +395,11 @@
       xyz="0 0 0" />
   </joint>
-<gazebo reference="lidar">
+  <link name="laser_frame"/>
+     <joint name="laser_frame_joint" type="fixed">
+        <parent link="lidar"/>
+        <child link="laser_frame"/>
+        <origin xyz="0 0 0" rpy="1.5707 0 0"/>
+    </joint>
+    <gazebo reference="laser_frame">
         <material>Gazebo/Grey</material>
         <sensor name="laser" type="gpu_lidar">
@@ -403,5 +409,5 @@
             <update_rate>10</update_rate>
             <topic>scan</topic>
-            <gz_frame_id>lidar</gz_frame_id>
+            <gz_frame_id>laser_frame</gz_frame_id>
             <lidar>
                 <scan>
